Commit message: feat: add slam package with configuration and launch files

File: src/bumperbot_description/urdf/bumperbot_core.xacro (robot description, xacro)
@@ -1,6 +1,12 @@
 <?xml version="1.0"?>
 <robot name="bumperbot" xmlns:xacro="http://ros.org/wiki/xacro">
-  <!-- Base Footprint -->
-  <link name="base_footprint"/>
+  <!-- BASE_FOOTPRINT LINK -->
+  <link name="base_footprint">
+  </link>
+  <joint name="base_footprint_joint" type="fixed">
+    <parent link="base_footprint"/>
+    <child link="base_link"/>
+    <origin xyz="0 0 0.033" rpy="0 0 0"/>
+  </joint>
   <!-- Base Link -->
   <link name="base_link">
@@ -25,9 +31,4 @@
     </collision>
   </link>
-  <joint name="base_joint" type="fixed">
-    <parent link="base_footprint"/>
-    <child link="base_link" />
-    <origin xyz="0 0 0.033" rpy="0 0 0"/>
-  </joint>
   <!-- Right Wheel -->
   <link name="wheel_right_link">

File: src/bumperbot_description/urdf/gazebo_control.xacro (robot description, xacro)
@@ -50,5 +50,5 @@
       <frame_id>odom</frame_id>
       <child_frame_id>base_footprint</child_frame_id>
-      <publish_odom_tf>true</publish_odom_tf>
+      <publish_odom_tf>false</publish_odom_tf>
     </plugin>
   </gazebo>
